File: hardware/Electronic-Load-XY-FZ25_ESP32C3-Circuit.kicad_pcb (KiCad board)
At the start: 2 copper layers, 91 x 31 mm, 19 parts, among them IC1 BD5330G, J1 Banana-Socket, J10 Conn_Terminal-Block_1x2, J2 Banana-Socket, J3 mech.-solder-pad_large, J4 mech.-solder-pad_large, J8 mech.-solder-pad, J9 Conn_1x4_PH, Q2 AO3416, U1 LiPO-Charge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

Commit message: Save
Parts:
- U3: value XIAO-ESP32C3 -> SEEEDUINO-XIAO-ESP32C3; footprint Marcus-PCB-Library:MOUDLE14P-SMD-2.54-21X17.8MM -> Marcus_Modules:SEEEDUINO-XIAO-ESP32C3
- renumbered 3.3V to J11, SW to J5, B+ to J6, 5.1V to J7
