File: hardware/Electronic-Load-XY-FZ25_ESP32C3-Circuit.kicad_sch (KiCad schematic)
At the start: 19 parts, among them IC1 BD5330G, J1 Banana-Socket, J10 Conn_Terminal-Block_1x2, J11 Conn_1x3_PH, J2 Banana-Socket, J3 mech.-solder-pad_large, J4 mech.-solder-pad_large, J5 Conn_1x2_PH, J6 Conn_1x2_PH, J7 Conn_1x3_PH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

Commit message: Save
Parts:
- removed U3: XIAO-ESP32C3, Marcus-PCB-Library:MOUDLE14P-SMD-2.54-21X17.8MM, symbol Marcus-PCB-Library:SEEEDUINO-XIAO-ESP32C3
- added U3: SEEEDUINO-XIAO-ESP32C3, Marcus_Modules:SEEEDUINO-XIAO-ESP32C3, symbol Marcus_Modules:SEEEDUINO-XIAO-ESP32C3
Connections:
- net +3.3V: now also U3.12 (3V3)
- net GND: now also U3.13 (GND)
- net at J9.3 (SCK), U2.3 (SCL): now also U3.6 (PA9_A5_D5_SCL)
- net at J9.4 (SDA), U2.4 (SDA): now also U3.5 (PA8_A4_D4_SDA)
- net at R1.2, R2.1: now also U3.1 (PA02_A0_D0)
- net at R3.1: now also U3.14 (5V)
Changed lines of the file:
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@@
-	)
-	(symbol
-		(lib_id "Marcus-PCB-Library:SEEEDUINO-XIAO-ESP32C3")
-		(at 186.69 51.435 0)
-		(unit 1)
-		(exclude_from_sim no)
-		(in_bom yes)
-		(on_board yes)
-		(dnp no)
-		(property "Reference" "U3"
-			(at 187.96 49.53 0)
-			(effects
-				(font
-					(size 1.27 1.27)
-				)
-			)
-		)
-		(property "Value" "XIAO-ESP32C3"
-			(at 204.47 49.53 0)
-			(effects
-				(font
-					(size 1.27 1.27)
-				)
-			)
-		)
-		(property "Footprint" "Marcus-PCB-Library:MOUDLE14P-SMD-2.54-21X17.8MM"
-			(at 184.785 36.195 0)
-			(effects
-				(font
-					(size 1.27 1.27)
-				)
-				(justify bottom)
-				(hide yes)
-			)
-		)
-		(property "Datasheet" ""
-			(at 186.69 51.435 0)
-			(effects
-				(font
-					(size 1.27 1.27)
-				)
-				(hide yes)
-			)
-		)
-		(property "Description" ""
-			(at 186.69 51.435 0)
-			(effects
-				(font
-					(size 1.27 1.27)
-				)
-				(hide yes)
-			)
-		)
-		(pin "14"
-		)
-		(pin "6"
-		)
-		(pin "2"
-		)
-		(pin "3"
-		)
-		(pin "4"
-		)
-		(pin "5"
-		)
-		(pin "7"
-		)
-		(pin "13"
-		)
-		(pin "12"
-		)
-		(pin "11"
-		)
-		(pin "10"
-		)
-		(pin "1"
-		)
-		(pin "9"
-		)
-		(pin "17"
-		)
-		(pin "8"
-		)
-		(pin "16"
-		)
-		(instances
-			(project ""
-				(path "/1594c9f4-f332-422d-b1bc-54e0c3ce6e4d"
-					(reference "U3")
-					(unit 1)
-				)
-			)
-		)
 	)
 	(symbol
@@
 					(unit 1)
 				)
+			)
+		)
+	)
+	(symbol
+		(lib_id "Marcus_Modules:SEEEDUINO-XIAO-ESP32C3")
+		(at 186.69 51.435 0)
+		(unit 1)
+		(exclude_from_sim no)
+		(in_bom yes)
+		(on_board yes)
+		(dnp no)
+		(fields_autoplaced yes)
+		(property "Reference" "U3"
+			(at 201.93 46.355 0)
+			(effects
+				(font
+					(size 1.27 1.27)
+				)
+			)
+		)
+		(property "Value" "SEEEDUINO-XIAO-ESP32C3"
+			(at 201.93 48.895 0)
+			(effects
+				(font
+					(size 1.27 1.27)
+				)
+			)
+		)
+		(property "Footprint" "Marcus_Modules:SEEEDUINO-XIAO-ESP32C3"
+			(at 206.375 50.165 0)
+			(effects
+				(font
+					(size 1.27 1.27)
+				)
+				(justify bottom)
+				(hide yes)
+			)
+		)
+		(property "Datasheet" ""
+			(at 208.28 65.405 0)
+			(effects
+				(font
+					(size 1.27 1.27)
+				)
+				(hide yes)
+			)
+		)
+		(property "Description" ""
+			(at 208.28 65.405 0)
+			(effects
+				(font
+					(size 1.27 1.27)
+				)
+				(hide yes)
+			)
+		)
+		(pin "1"
+		)
+		(pin "4"
+		)
+		(pin "2"
+		)
+		(pin "3"
+		)
+		(pin "7"
+		)
+		(pin "11"
+		)
+		(pin "14"
+		)
+		(pin "9"
+		)
+		(pin "8"
+		)
+		(pin "16"
+		)
+		(pin "17"
+		)
+		(pin "5"
+		)
+		(pin "6"
+		)
+		(pin "13"
+		)
+		(pin "12"
+		)
+		(pin "10"
+		)
+		(instances
+			(project ""
+				(path "/1594c9f4-f332-422d-b1bc-54e0c3ce6e4d"
+					(reference "U3")
+					(unit 1)
+				)
